File: hardware/PCB/ZAEMON.kicad_sch (KiCad schematic)
At the start: 8 parts, among them J3 Servo_motor_power_left, J4 Servo_motor_power_right, J5 ESP32_power, U1 DEVKIT_V1_ESP32-WROOM-32

Commit message: feat: update ZAEMON PCB design
Parts:
- removed Servo_Left_Buck, Servo_Right_Buck: MP1584_DC-DC, Package_SO:SOIC-8_3.9x4.9mm_P1.27mm, symbol Custom_board:MP1584_DC-DC
- added C3, C4: 1000uF, Capacitor_THT:CP_Radial_D10.0mm_P5.00mm, symbol Device:C
- added J1: Driver_Right_Input, Connector_PinHeader_2.54mm:PinHeader_2x05_P2.54mm_Vertical, symbol Connector_Generic:Conn_02x05_Odd_Even
- added J10: Servo_Left, Connector_PinHeader_2.54mm:PinHeader_1x03_P2.54mm_Vertical, symbol Connector:Conn_01x03_Pin
- added J11: Servo_Right, Connector_PinHeader_2.54mm:PinHeader_1x03_P2.54mm_Vertical, symbol Connector:Conn_01x03_Pin
- added J12: MPU6050, Connector_PinHeader_2.54mm:PinHeader_1x08_P2.54mm_Vertical, symbol Connector:Conn_01x08_Pin
- added J2: Driver_Left_Input, Connector_PinHeader_2.54mm:PinHeader_2x05_P2.54mm_Vertical, symbol Connector_Generic:Conn_02x05_Odd_Even
- added J6: Driver_Right_Output, Connector_PinHeader_2.54mm:PinHeader_1x03_P2.54mm_Vertical, symbol Connector:Conn_01x03_Socket
- added J7: Driver_Left_Output, Connector_PinHeader_2.54mm:PinHeader_1x03_P2.54mm_Vertical, symbol Connector:Conn_01x03_Socket
- added J8: Right_Leg, Connector_PinHeader_2.54mm:PinHeader_1x07_P2.54mm_Vertical, symbol Connector:Conn_01x07_Socket
- added J9: Left_Leg, Connector_PinHeader_2.54mm:PinHeader_1x07_P2.54mm_Vertical, symbol Connector:Conn_01x07_Socket
- added U2, U3: MP1584_DC-DC, symbol Custom_board:MP1584_DC-DC
- C1: value C -> 470uF; footprint (none) -> Capacitor_THT:CP_Radial_D10.0mm_P5.00mm
- C2: value C -> 100nF; footprint (none) -> Capacitor_THT:C_Disc_D5.0mm_W2.5mm_P5.00mm
- J3, J4, J5: footprint Package_SON:WSON-8-1EP_6x5mm_P1.27mm_EP3.4x4mm -> TerminalBlock_Phoenix:TerminalBlock_Phoenix_MKDS-1,5-2-5.08_1x02_P5.08mm_Horizontal
Connections:
- net 5V_BEC_GND is gone; now on net GND: C1.2, C2.2, J5.2 (Pin_2)
- net 5V_BEC: now also C1.1, C2.1, U1.30 (VIN), J12.1 (Pin_1), J8.1 (Pin_1), J9.1 (Pin_1)
- net GND: now also J1.9 (Pin_9), J12.2 (Pin_2), J2.9 (Pin_9), J8.2 (Pin_2), J9.2 (Pin_2)
- net Servo_left_negative_PDB: now also U2.2 (IN-)
- net Servo_left_positive_PDB: now also U2.1 (IN+)
- net Servo_right_negative_PDB: now also U3.2 (IN-)
- net Servo_right_positive_PDB: now also U3.1 (IN+)
- net Driver_Left_EN: now reaches U1.1 (3V3)
- net Driver_Left_EN: now also J1.1 (Pin_1), J2.1 (Pin_1)
- net I2C0_SDA: now reaches U1.11 (D21)
- net I2C0_SDA: now also J12.4 (Pin_4), J8.3 (Pin_3)
- net I2C0_SCL: now reaches U1.14 (D22)
- net I2C0_SCL: now also J12.3 (Pin_3), J8.4 (Pin_4)
- net Driver_Right_IN1: now reaches U1.15 (D23)
- net Driver_Right_IN1: now also J1.7 (Pin_7)
- net Driver_Right_nFAULT: now reaches U1.18 (VN)
- net Driver_Right_nFAULT: now also J1.2 (Pin_2)
- net MPU6050_INT: now reaches U1.19 (D34)
- net MPU6050_INT: now also J12.8 (Pin_8)
- net Driver_Left_nFAULT: now reaches U1.20 (D35)
- net Driver_Left_nFAULT: now also J2.2 (Pin_2)
- net I2C1_SDA: now reaches U1.21 (D32)
- net I2C1_SDA: now also J9.4 (Pin_4)
- net I2C1_SCL: now reaches U1.22 (D33)
- net I2C1_SCL: now also J9.3 (Pin_3)
- net Driver_Right_IN2: now reaches U1.23 (D25)
- net Driver_Right_IN2: now also J1.5 (Pin_5)
- net Driver_Right_IN3: now reaches U1.24 (D26)
- net Driver_Right_IN3: now also J1.3 (Pin_3)
- net nSLEEP: now reaches U1.25 (D27)
- net nSLEEP: now also J1.4 (Pin_4), J2.4 (Pin_4)
- net Servo_Right_data: now reaches U1.26 (D14)
- net Servo_Right_data: now also J11.3 (Pin_3)
- net Servo_Left_data: now reaches U1.28 (D13)
- net Servo_Left_data: now also J10.3 (Pin_3)
- net Driver_Left_IN1: now reaches U1.6 (RX2)
- net Driver_Left_IN1: now also J2.7 (Pin_7)
- net Driver_Left_IN2: now reaches U1.7 (TX2)
- net Driver_Left_IN2: now also J2.5 (Pin_5)
- net Driver_Left_IN3: now reaches U1.9 (D18)
- net Driver_Left_IN3: now also J2.3 (Pin_3)
- new net Left_IN1: J7.3 (Pin_3), J9.7 (Pin_7)
- new net Left_IN2: J7.2 (Pin_2), J9.6 (Pin_6)
- new net Left_IN3: J7.1 (Pin_1), J9.5 (Pin_5)
- new net Right_IN1: J6.3 (Pin_3), J8.7 (Pin_7)
- new net Right_IN2: J6.2 (Pin_2), J8.6 (Pin_6)
- new net Right_IN3: J6.1 (Pin_1), J8.5 (Pin_5)
- new net Servo_left_negative: C3.2, J10.1 (Pin_1), U2. (OUT-)
- new net Servo_left_positive: C3.1, J10.2 (Pin_2), U2. (OUT-)
- new net Servo_right_negative: C4.2, J11.1 (Pin_1), U3. (OUT-)
- new net Servo_right_positive: C4.1, J11.2 (Pin_2), U3. (OUT-)
- no-connect marks 0 -> 19
Other:
- note removed: "PDB to Buck to Servo"
- moved on the sheet: C1, C2, U1
